File: hw/MIC_module.sch (EAGLE design)
At the start: 35 parts, among them J1 GROVE-4P-2.0-3470130P1, J2 GROVE-4P-2.0-3470130P1

Commit message: added USB port
Parts:
- added J4: MICRO-USB-5P-340015001, OPL Eagle Library:MICRO-USB-5P-340015001
- added R11, R14: 22, rcl:R-EU_R0603
- added R6: 100k, rcl:R-EU_R0603
- added R8: 1k5, rcl:R-EU_R0603
Connections:
- new net N$3: J4.DM, R11.2
- new net N$32: J4.DP, R14.2, R8.2
- new net N$5: J4.ID, R6.2
- new net USB_N: R11.1, U$6.PA11
- new net USB_P: R14.1, U$6.PA12
- new net USB_VBUS: J4.VCC
- net +3V3: now also R8.1
- net GND: now also J4.GND@1, J4.GND@2, J4.GND@3, R6.1
Other:
- note added: "USB INTERFACE"
Changed lines of the file:
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@@
 <part name="C15" library="rcl" deviceset="C-EU" device="C0603" value="15p"/>
 <part name="GND27" library="supply1" deviceset="GND" device=""/>
+<part name="GND38" library="supply1" deviceset="GND" device=""/>
+<part name="R11" library="rcl" deviceset="R-EU_" device="R0603" value="22"/>
+<part name="R14" library="rcl" deviceset="R-EU_" device="R0603" value="22"/>
+<part name="R6" library="rcl" deviceset="R-EU_" device="R0603" value="100k"/>
+<part name="GND28" library="supply1" deviceset="GND" device=""/>
+<part name="R8" library="rcl" deviceset="R-EU_" device="R0603" value="1k5"/>
+<part name="+3V14" library="supply1" deviceset="+3V3" device=""/>
+<part name="J4" library="OPL Eagle Library" deviceset="MICRO-USB-5P" device="-340015001"/>
 </parts>
 <sheets>
@@
 <wire x1="55.88" y1="5.08" x2="55.88" y2="43.18" width="0.1524" layer="94"/>
 <text x="58.42" y="38.1" size="2.54" layer="94">R2P BUS</text>
+<wire x1="160.02" y1="73.66" x2="220.98" y2="73.66" width="0.1524" layer="94"/>
+<wire x1="220.98" y1="73.66" x2="220.98" y2="22.86" width="0.1524" layer="94"/>
+<wire x1="220.98" y1="22.86" x2="160.02" y2="22.86" width="0.1524" layer="94"/>
+<wire x1="160.02" y1="22.86" x2="160.02" y2="73.66" width="0.1524" layer="94"/>
+<text x="162.56" y="68.58" size="2.54" layer="94">USB INTERFACE</text>
 </plain>
 <instances>
@@
 <instance part="C15" gate="G$1" x="195.58" y="149.86"/>
 <instance part="GND27" gate="1" x="195.58" y="142.24"/>
+<instance part="GND38" gate="1" x="198.12" y="30.48"/>
+<instance part="R11" gate="G$1" x="180.34" y="50.8"/>
+<instance part="R14" gate="G$1" x="180.34" y="43.18"/>
+<instance part="R6" gate="G$1" x="190.5" y="38.1" rot="R90"/>
+<instance part="GND28" gate="1" x="190.5" y="30.48"/>
+<instance part="R8" gate="G$1" x="198.12" y="63.5" rot="R180"/>
+<instance part="+3V14" gate="G$1" x="205.74" y="71.12"/>
+<instance part="J4" gate="USB" x="208.28" y="45.72" rot="MR0"/>
 </instances>
 <busses>
@@
 <pinref part="C15" gate="G$1" pin="2"/>
 <pinref part="GND27" gate="1" pin="GND"/>
+</segment>
+<segment>
+<pinref part="GND38" gate="1" pin="GND"/>
+<wire x1="198.12" y1="33.02" x2="198.12" y2="40.64" width="0.1524" layer="91"/>
+<wire x1="208.28" y1="33.02" x2="205.74" y2="33.02" width="0.1524" layer="91"/>
+<wire x1="205.74" y1="33.02" x2="203.2" y2="33.02" width="0.1524" layer="91"/>
+<wire x1="203.2" y1="33.02" x2="200.66" y2="33.02" width="0.1524" layer="91"/>
+<wire x1="200.66" y1="33.02" x2="198.12" y2="33.02" width="0.1524" layer="91"/>
+<junction x="198.12" y="33.02"/>
+<pinref part="J4" gate="USB" pin="GND@1"/>
+<pinref part="J4" gate="USB" pin="GND@2"/>
+<wire x1="208.28" y1="33.02" x2="218.44" y2="33.02" width="0.1524" layer="91"/>
+<wire x1="218.44" y1="33.02" x2="218.44" y2="44.45" width="0.1524" layer="91"/>
+<pinref part="J4" gate="USB" pin="GND@3"/>
+<wire x1="218.44" y1="44.45" x2="218.44" y2="46.99" width="0.1524" layer="91"/>
+<junction x="218.44" y="44.45"/>
+</segment>
+<segment>
+<pinref part="R6" gate="G$1" pin="1"/>
+<pinref part="GND28" gate="1" pin="GND"/>
 </segment>
 </net>
@@
 <wire x1="180.34" y1="195.58" x2="180.34" y2="198.12" width="0.1524" layer="91"/>
 </segment>
+<segment>
+<pinref part="R8" gate="G$1" pin="1"/>
+<wire x1="203.2" y1="63.5" x2="205.74" y2="63.5" width="0.1524" layer="91"/>
+<wire x1="205.74" y1="63.5" x2="205.74" y2="68.58" width="0.1524" layer="91"/>
+<pinref part="+3V14" gate="G$1" pin="+3V3"/>
+</segment>
 </net>
 <net name="JTMS" class="0">
@@
 </segment>
 </net>
+<net name="USB_VBUS" class="0">
+<segment>
+<wire x1="198.12" y1="50.8" x2="195.58" y2="50.8" width="0.1524" layer="91"/>
+<label x="177.8" y="58.42" size="1.778" layer="95" rot="MR0"/>
+<wire x1="195.58" y1="50.8" x2="195.58" y2="58.42" width="0.1524" layer="91"/>
+<wire x1="195.58" y1="58.42" x2="177.8" y2="58.42" width="0.1524" layer="91"/>
+<pinref part="J4" gate="USB" pin="VCC"/>
+</segment>
+</net>
+<net name="USB_N" class="0">
+<segment>
+<pinref part="R11" gate="G$1" pin="1"/>
+<wire x1="175.26" y1="50.8" x2="172.72" y2="50.8" width="0.1524" layer="91"/>
+<label x="172.72" y="50.8" size="1.778" layer="95" rot="MR0"/>
+</segment>
+<segment>
+<pinref part="U$6" gate="G$1" pin="PA11"/>
+<wire x1="58.42" y1="177.8" x2="58.42" y2="175.26" width="0.1524" layer="91"/>
+<label x="58.42" y="175.26" size="1.778" layer="95" rot="MR270"/>
+</segment>
+</net>
+<net name="USB_P" class="0">
+<segment>
+<pinref part="R14" gate="G$1" pin="1"/>
+<wire x1="175.26" y1="43.18" x2="172.72" y2="43.18" width="0.1524" layer="91"/>
+<label x="172.72" y="43.18" size="1.778" layer="95" rot="MR0"/>
+</segment>
+<segment>
+<pinref part="U$6" gate="G$1" pin="PA12"/>
+<wire x1="60.96" y1="177.8" x2="60.96" y2="175.26" width="0.1524" layer="91"/>
+<label x="60.96" y="175.26" size="1.778" layer="95" rot="MR270"/>
+</segment>
+</net>
+<net name="N$3" class="0">
+<segment>
+<wire x1="198.12" y1="48.26" x2="187.96" y2="48.26" width="0.1524" layer="91"/>
+<wire x1="187.96" y1="48.26" x2="187.96" y2="50.8" width="0.1524" layer="91"/>
+<pinref part="R11" gate="G$1" pin="2"/>
+<wire x1="187.96" y1="50.8" x2="185.42" y2="50.8" width="0.1524" layer="91"/>
+<pinref part="J4" gate="USB" pin="DM"/>
+</segment>
+</net>
+<net name="N$32" class="0">
+<segment>
+<wire x1="198.12" y1="45.72" x2="190.5" y2="45.72" width="0.1524" layer="91"/>
+<wire x1="190.5" y1="45.72" x2="187.96" y2="45.72" width="0.1524" layer="91"/>
+<wire x1="187.96" y1="45.72" x2="187.96" y2="43.18" width="0.1524" layer="91"/>
+<pinref part="R14" gate="G$1" pin="2"/>
+<wire x1="187.96" y1="43.18" x2="185.42" y2="43.18" width="0.1524" layer="91"/>
+<pinref part="R8" gate="G$1" pin="2"/>
+<wire x1="193.04" y1="63.5" x2="190.5" y2="63.5" width="0.1524" layer="91"/>
+<wire x1="190.5" y1="63.5" x2="190.5" y2="45.72" width="0.1524" layer="91"/>
+<junction x="190.5" y="45.72"/>
+<pinref part="J4" gate="USB" pin="DP"/>
+</segment>
+</net>
+<net name="N$5" class="0">
+<segment>
+<pinref part="R6" gate="G$1" pin="2"/>
+<wire x1="190.5" y1="43.18" x2="198.12" y2="43.18" width="0.1524" layer="91"/>
+<pinref part="J4" gate="USB" pin="ID"/>
+</segment>
+</net>

Commit message: fixed led polarity
Connections:
- net GND: now also LED1.C; no longer LED1.A
- net N$4: now also LED1.A; no longer LED1.C
Other:
- moved on the sheet: LED1
Changed lines of the file:
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@@
 <instance part="C7" gate="G$1" x="124.46" y="71.12"/>
 <instance part="GND22" gate="1" x="124.46" y="63.5"/>
-<instance part="LED1" gate="G$1" x="22.86" y="114.3" rot="R180"/>
+<instance part="LED1" gate="G$1" x="22.86" y="114.3"/>
 <instance part="R1" gate="G$1" x="22.86" y="127" rot="R90"/>
 <instance part="GND16" gate="1" x="81.28" y="10.16"/>
@@
 <instance part="FRAME1" gate="G$1" x="0" y="0"/>
 <instance part="FRAME1" gate="G$2" x="287.02" y="0"/>
-<instance part="GND13" gate="1" x="22.86" y="109.22"/>
+<instance part="GND13" gate="1" x="22.86" y="104.14"/>
 <instance part="SOT1" gate="G$1" x="93.98" y="68.58"/>
 <instance part="U$1" gate="A" x="27.94" y="22.86"/>
@@
 </segment>
 <segment>
-<pinref part="LED1" gate="G$1" pin="A"/>
 <pinref part="GND13" gate="1" pin="GND"/>
+<wire x1="22.86" y1="106.68" x2="22.86" y2="109.22" width="0.1524" layer="91"/>
+<pinref part="LED1" gate="G$1" pin="C"/>
 </segment>
 <segment>
@@
 <segment>
 <pinref part="R1" gate="G$1" pin="1"/>
-<pinref part="LED1" gate="G$1" pin="C"/>
-<wire x1="22.86" y1="119.38" x2="22.86" y2="121.92" width="0.1524" layer="91"/>
-</segment>
-</net>
+<wire x1="22.86" y1="116.84" x2="22.86" y2="121.92" width="0.1524" layer="91"/>
+<pinref part="LED1" gate="G$1" pin="A"/>
+</segment>
+</net>
